File: BMS.kicad_pcb (KiCad board)
At the start: 2 copper layers, 14 parts, among them Q1 BSC028N06LS3, U1 BQ76920PW, U2 453-00001R

Commit message: Added Todo
Parts:
- added C1: 1u, Capacitor_SMD:C_0805_2012Metric_Pad1.18x1.45mm_HandSolder, F.Cu at (116.7, 84.3)
- added C10: 100n, Capacitor_SMD:C_0805_2012Metric_Pad1.18x1.45mm_HandSolder, F.Cu at (126.3, 87.3)
- added C11: 4u7, Capacitor_SMD:C_0805_2012Metric_Pad1.18x1.45mm_HandSolder, F.Cu at (126.3, 90.4)
- added C12: 1u, Capacitor_SMD:C_0805_2012Metric_Pad1.18x1.45mm_HandSolder, F.Cu at (126.3, 93.4)
- added C13: 10n, Capacitor_SMD:C_0805_2012Metric_Pad1.18x1.45mm_HandSolder, F.Cu at (33.1, 41.9)
- added C14: 100u, Capacitor_SMD:C_0805_2012Metric_Pad1.18x1.45mm_HandSolder, F.Cu at (46.7, 82.8)
- added C15: 220u, Capacitor_SMD:C_0805_2012Metric_Pad1.18x1.45mm_HandSolder, F.Cu at (46.7, 85.8)
- added C16: 10n, Capacitor_SMD:C_0805_2012Metric_Pad1.18x1.45mm_HandSolder, F.Cu at (46.7, 88.8)
- added C17: 4u7, Capacitor_SMD:C_0805_2012Metric_Pad1.18x1.45mm_HandSolder, F.Cu at (33.1, 44.9)
- added C18: 22u, Capacitor_SMD:C_0805_2012Metric_Pad1.18x1.45mm_HandSolder, F.Cu at (33.1, 47.9)
- added C19: 100n, Capacitor_SMD:C_0805_2012Metric_Pad1.18x1.45mm_HandSolder, F.Cu at (33.1, 50.9)
- added C2: 1u, Capacitor_SMD:C_0805_2012Metric_Pad1.18x1.45mm_HandSolder, F.Cu at (116.7, 87.3)
- added C20: 22u, Capacitor_SMD:C_0805_2012Metric_Pad1.18x1.45mm_HandSolder, F.Cu at (33.1, 54.0)
- added C21: 100n, Capacitor_SMD:C_0805_2012Metric_Pad1.18x1.45mm_HandSolder, F.Cu at (26.3, 41.9)
- added C22: 100u, Capacitor_SMD:C_0805_2012Metric_Pad1.18x1.45mm_HandSolder, F.Cu at (26.3, 44.9)
- added C23: 22u, Capacitor_SMD:C_0805_2012Metric_Pad1.18x1.45mm_HandSolder, F.Cu at (33.1, 57.0)
- added C24: 100n, Capacitor_SMD:C_0805_2012Metric_Pad1.18x1.45mm_HandSolder, F.Cu at (37.9, 41.9)
- added C25: 10n, Capacitor_SMD:C_0805_2012Metric_Pad1.18x1.45mm_HandSolder, F.Cu at (37.9, 44.9)
- added C26: 4u7, Capacitor_SMD:C_0805_2012Metric_Pad1.18x1.45mm_HandSolder, F.Cu at (37.9, 47.9)
- added C27: 22u, Capacitor_SMD:C_0805_2012Metric_Pad1.18x1.45mm_HandSolder, F.Cu at (37.9, 50.9)
- added C28: 22u, Capacitor_SMD:C_0805_2012Metric_Pad1.18x1.45mm_HandSolder, F.Cu at (79.5, 78.1)
- added C29: 22u, Capacitor_SMD:C_0805_2012Metric_Pad1.18x1.45mm_HandSolder, F.Cu at (79.5, 81.1)
- added C3: 1u, Capacitor_SMD:C_0805_2012Metric_Pad1.18x1.45mm_HandSolder, F.Cu at (116.7, 90.4)
- added C30: 22u, Capacitor_SMD:C_0805_2012Metric_Pad1.18x1.45mm_HandSolder, F.Cu at (79.5, 84.1)
- added C31: 100n, Capacitor_SMD:C_0805_2012Metric_Pad1.18x1.45mm_HandSolder, F.Cu at (79.5, 87.1)
- added C32: 100n, Capacitor_SMD:C_0805_2012Metric_Pad1.18x1.45mm_HandSolder, F.Cu at (79.5, 90.1)
- added C33: 22u, Capacitor_SMD:C_0805_2012Metric_Pad1.18x1.45mm_HandSolder, F.Cu at (37.9, 54.0)
- added C34: 100n, Capacitor_SMD:C_0805_2012Metric_Pad1.18x1.45mm_HandSolder, F.Cu at (37.9, 57.0)
- added C35: 10n, Capacitor_SMD:C_0805_2012Metric_Pad1.18x1.45mm_HandSolder, F.Cu at (42.7, 41.9)
- added C36: 4u7, Capacitor_SMD:C_0805_2012Metric_Pad1.18x1.45mm_HandSolder, F.Cu at (42.7, 44.9)
- added C37: 22u, Capacitor_SMD:C_0805_2012Metric_Pad1.18x1.45mm_HandSolder, F.Cu at (42.7, 47.9)
- added C38: 100n, Capacitor_SMD:C_0805_2012Metric_Pad1.18x1.45mm_HandSolder, F.Cu at (79.5, 93.1)
- added C39: 10n, Capacitor_SMD:C_0805_2012Metric_Pad1.18x1.45mm_HandSolder, F.Cu at (84.3, 78.1)
- added C4: 1u, Capacitor_SMD:C_0805_2012Metric_Pad1.18x1.45mm_HandSolder, F.Cu at (116.7, 93.4)
- added C40: 10n, Capacitor_SMD:C_0805_2012Metric_Pad1.18x1.45mm_HandSolder, F.Cu at (84.3, 81.1)
- added C41: 10n, Capacitor_SMD:C_0805_2012Metric_Pad1.18x1.45mm_HandSolder, F.Cu at (84.3, 84.1)
- added C42: 4u7, Capacitor_SMD:C_0805_2012Metric_Pad1.18x1.45mm_HandSolder, F.Cu at (84.3, 87.1)
- added C43: 4u7, Capacitor_SMD:C_0805_2012Metric_Pad1.18x1.45mm_HandSolder, F.Cu at (84.3, 90.1)
- added C44: 4u7, Capacitor_SMD:C_0805_2012Metric_Pad1.18x1.45mm_HandSolder, F.Cu at (84.3, 93.1)
- added C45: 22u, Capacitor_SMD:C_0805_2012Metric_Pad1.18x1.45mm_HandSolder, F.Cu at (89.2, 78.1)
- added C46: 22u, Capacitor_SMD:C_0805_2012Metric_Pad1.18x1.45mm_HandSolder, F.Cu at (89.2, 81.1)
- added C47: 22u, Capacitor_SMD:C_0805_2012Metric_Pad1.18x1.45mm_HandSolder, F.Cu at (89.2, 84.1)
- added C5: 1u, Capacitor_SMD:C_0805_2012Metric_Pad1.18x1.45mm_HandSolder, F.Cu at (121.5, 84.3)
- added C6: 1u, Capacitor_SMD:C_0805_2012Metric_Pad1.18x1.45mm_HandSolder, F.Cu at (121.5, 87.3)
- added C7: 10u, Capacitor_SMD:C_0805_2012Metric_Pad1.18x1.45mm_HandSolder, F.Cu at (121.5, 90.4)
- added C8: 100n, Capacitor_SMD:C_0805_2012Metric_Pad1.18x1.45mm_HandSolder, F.Cu at (121.5, 93.4)
- added C9: 100n, Capacitor_SMD:C_0805_2012Metric_Pad1.18x1.45mm_HandSolder, F.Cu at (126.3, 84.3)
- added D1: 1N5822, Diode_THT:D_DO-201AD_P15.24mm_Horizontal, F.Cu at (33.1, 77.9)
- added IC1: AOZ2261NQI-11, LIB_AOZ2261NQI-11:AOZ2261NQI11, F.Cu at (117.6, 100.5)
- added IC2: AOZ2261NQI-11, LIB_AOZ2261NQI-11:AOZ2261NQI11, F.Cu at (108.4, 100.5)
- added IC2: LM2596DSADJG, LIB_LM2596DSADJG:LM2596DSADJG, F.Cu at (37.5, 90.7)
- added IC3: AOZ2261NQI-11, LIB_AOZ2261NQI-11:AOZ2261NQI11, F.Cu at (48.7, 61.7)
- added IC4: AOZ2261NQI-11, LIB_AOZ2261NQI-11:AOZ2261NQI11, F.Cu at (73.5, 80.2)
- added IC5: AOZ2261NQI-11, LIB_AOZ2261NQI-11:AOZ2261NQI11, F.Cu at (48.7, 68.9)
- added IC6: AOZ2261NQI-11, LIB_AOZ2261NQI-11:AOZ2261NQI11, F.Cu at (73.5, 87.4)
- added IC7: AOZ2261NQI-11, LIB_AOZ2261NQI-11:AOZ2261NQI11, F.Cu at (73.5, 94.6)
- added J1: Conn_01x05_Pin, Connector_JST:JST_XH_B5B-XH-A_1x05_P2.50mm_Vertical, F.Cu at (117.7, 78.4)
- added J10: XT90PB-F, XT90PB-F:XT90PBF, F.Cu at (195.0, 109.5)
- added J11: XT90PB-F, XT90PB-F:XT90PBF, F.Cu at (195.0, 123.5)
- added J12: XT90PB-F, XT90PB-F:XT90PBF, F.Cu at (171.0, 39.0)
- added J2: XT90PB-F, XT90PB-F:XT90PBF, F.Cu at (117.4, 122.5)
- added J3: Conn_01x02_Pin, Connector_PinHeader_2.54mm:PinHeader_1x02_P2.54mm_Vertical, F.Cu at (136.0, 63.3)
- added J4: Conn_01x03_Pin, Connector_PinHeader_2.54mm:PinHeader_1x03_P2.54mm_Vertical, F.Cu at (131.5, 63.3)
- added J5: XT90PB-F, XT90PB-F:XT90PBF, F.Cu at (195.5, 39.2)
- added J6: XT90PB-F, XT90PB-F:XT90PBF, F.Cu at (195.5, 53.2)
- added J7: XT90PB-F, XT90PB-F:XT90PBF, F.Cu at (195.5, 67.2)
- added J8: XT90PB-F, XT90PB-F:XT90PBF, F.Cu at (195.5, 81.2)
- added J9: XT90PB-F, XT90PB-F:XT90PBF, F.Cu at (195.5, 95.2)
- added L1: 33u, Inductor_SMD:L_0805_2012Metric_Pad1.15x1.40mm_HandSolder, F.Cu at (46.7, 91.8)
- added L2: 1u, Inductor_SMD:L_0805_2012Metric_Pad1.15x1.40mm_HandSolder, F.Cu at (47.5, 41.9)
- added L3: 1u, Inductor_SMD:L_0805_2012Metric_Pad1.15x1.40mm_HandSolder, F.Cu at (47.5, 44.8)
- added L4: 1u, Inductor_SMD:L_0805_2012Metric_Pad1.15x1.40mm_HandSolder, F.Cu at (79.5, 96.1)
- added L5: 1u, Inductor_SMD:L_0805_2012Metric_Pad1.15x1.40mm_HandSolder, F.Cu at (47.5, 47.8)
- added L6: 1u, Inductor_SMD:L_0805_2012Metric_Pad1.15x1.40mm_HandSolder, F.Cu at (79.5, 99.0)
- added L7: 1u, Inductor_SMD:L_0805_2012Metric_Pad1.15x1.40mm_HandSolder, F.Cu at (79.5, 102.0)
- added Q2: IRLB3813PBF, digikey-footprints:TO-220-3, F.Cu at (131.9, 85.9)
- added R1: 100, Resistor_SMD:R_0805_2012Metric_Pad1.20x1.40mm_HandSolder, F.Cu at (107.1, 76.5)
- added R10: 1M, Resistor_SMD:R_0805_2012Metric_Pad1.20x1.40mm_HandSolder, F.Cu at (111.9, 76.5)
- added R11: 100, Resistor_SMD:R_0805_2012Metric_Pad1.20x1.40mm_HandSolder, F.Cu at (111.9, 79.5)
- added R12: 100, Resistor_SMD:R_0805_2012Metric_Pad1.20x1.40mm_HandSolder, F.Cu at (111.9, 82.4)
- added R13: 10k, Resistor_SMD:R_0805_2012Metric_Pad1.20x1.40mm_HandSolder, F.Cu at (111.9, 85.4)
- added R15: 4k7, Resistor_SMD:R_0805_2012Metric_Pad1.20x1.40mm_HandSolder, F.Cu at (111.9, 88.3)
- added R2: 100, Resistor_SMD:R_0805_2012Metric_Pad1.20x1.40mm_HandSolder, F.Cu at (107.1, 79.5)
- added R24: 3k1, Resistor_SMD:R_0805_2012Metric_Pad1.20x1.40mm_HandSolder, F.Cu at (46.7, 94.7)
- added R25: 1k, Resistor_SMD:R_0805_2012Metric_Pad1.20x1.40mm_HandSolder, F.Cu at (46.7, 97.7)
- added R26: 100k, Resistor_SMD:R_0805_2012Metric_Pad1.20x1.40mm_HandSolder, F.Cu at (47.5, 50.7)
- added R27: 100k, Resistor_SMD:R_0805_2012Metric_Pad1.20x1.40mm_HandSolder, F.Cu at (47.5, 53.7)
- added R28: 190k, Resistor_SMD:R_0805_2012Metric_Pad1.20x1.40mm_HandSolder, F.Cu at (47.5, 56.6)
- added R29: 10k, Resistor_SMD:R_0805_2012Metric_Pad1.20x1.40mm_HandSolder, F.Cu at (52.3, 41.9)
- added R3: 100, Resistor_SMD:R_0805_2012Metric_Pad1.20x1.40mm_HandSolder, F.Cu at (107.1, 82.4)
- added R30: 100k, Resistor_SMD:R_0805_2012Metric_Pad1.20x1.40mm_HandSolder, F.Cu at (52.3, 44.8)
- added R31: 100k, Resistor_SMD:R_0805_2012Metric_Pad1.20x1.40mm_HandSolder, F.Cu at (52.3, 47.8)
- added R32: 140k, Resistor_SMD:R_0805_2012Metric_Pad1.20x1.40mm_HandSolder, F.Cu at (52.3, 50.7)
- added R33: 10k, Resistor_SMD:R_0805_2012Metric_Pad1.20x1.40mm_HandSolder, F.Cu at (52.3, 53.7)
- added R34: 100k, Resistor_SMD:R_0805_2012Metric_Pad1.20x1.40mm_HandSolder, F.Cu at (79.5, 105.0)
- added R35: 100k, Resistor_SMD:R_0805_2012Metric_Pad1.20x1.40mm_HandSolder, F.Cu at (79.5, 107.9)
- added R36: 100k, Resistor_SMD:R_0805_2012Metric_Pad1.20x1.40mm_HandSolder, F.Cu at (79.5, 110.8)
- added R37: 100k, Resistor_SMD:R_0805_2012Metric_Pad1.20x1.40mm_HandSolder, F.Cu at (84.2, 96.1)
- added R38: 100k, Resistor_SMD:R_0805_2012Metric_Pad1.20x1.40mm_HandSolder, F.Cu at (52.3, 56.6)
- added R39: 100k, Resistor_SMD:R_0805_2012Metric_Pad1.20x1.40mm_HandSolder, F.Cu at (57.0, 41.9)
- added R4: 100, Resistor_SMD:R_0805_2012Metric_Pad1.20x1.40mm_HandSolder, F.Cu at (107.1, 85.4)
- added R40: 75k, Resistor_SMD:R_0805_2012Metric_Pad1.20x1.40mm_HandSolder, F.Cu at (57.0, 44.8)
- added R41: 10k, Resistor_SMD:R_0805_2012Metric_Pad1.20x1.40mm_HandSolder, F.Cu at (57.0, 47.8)
- added R42: 100k, Resistor_SMD:R_0805_2012Metric_Pad1.20x1.40mm_HandSolder, F.Cu at (84.2, 99.0)
- added R43: 100k, Resistor_SMD:R_0805_2012Metric_Pad1.20x1.40mm_HandSolder, F.Cu at (84.2, 102.0)
- added R44: 190k, Resistor_SMD:R_0805_2012Metric_Pad1.20x1.40mm_HandSolder, F.Cu at (84.2, 105.0)
- added R45: 10k, Resistor_SMD:R_0805_2012Metric_Pad1.20x1.40mm_HandSolder, F.Cu at (84.2, 107.9)
- added R46: 140k, Resistor_SMD:R_0805_2012Metric_Pad1.20x1.40mm_HandSolder, F.Cu at (84.2, 110.8)
- added R47: 10k, Resistor_SMD:R_0805_2012Metric_Pad1.20x1.40mm_HandSolder, F.Cu at (89.0, 96.1)
- added R48: 75k, Resistor_SMD:R_0805_2012Metric_Pad1.20x1.40mm_HandSolder, F.Cu at (89.0, 99.0)
- added R49: 10k, Resistor_SMD:R_0805_2012Metric_Pad1.20x1.40mm_HandSolder, F.Cu at (89.0, 102.0)
- added R5: 100, Resistor_SMD:R_0805_2012Metric_Pad1.20x1.40mm_HandSolder, F.Cu at (107.1, 88.3)
- added R6: 100, Resistor_SMD:R_0805_2012Metric_Pad1.20x1.40mm_HandSolder, F.Cu at (107.1, 91.3)
- added R7: 4k7', Resistor_SMD:R_0805_2012Metric_Pad1.20x1.40mm_HandSolder, F.Cu at (125.5, 98.3)
- added R8: 4k7, Resistor_SMD:R_0805_2012Metric_Pad1.20x1.40mm_HandSolder, F.Cu at (125.5, 101.3)
- moved R18 19.3 mm to (106.4, 42.3)
- moved R23 19.3 mm to (106.4, 50.5)
- moved U1 19.3 mm to (133.1, 48.4)
- moved Q1 19.3 mm to (101.1, 58.0)
- moved R16 19.3 mm to (95.7, 42.3)
- moved R17 19.3 mm to (101.1, 42.3)
- moved R19 19.3 mm to (85.1, 50.5)
- moved R21 19.3 mm to (95.7, 50.5)
- moved R22 19.3 mm to (101.1, 50.5)
- moved R9 19.3 mm to (85.1, 42.3)
- moved S1 19.3 mm to (87.1, 56.5)
- moved U2 19.3 mm to (117.8, 52.2)
- moved R14 17.0 mm to (85.0, 26.0)
- moved R20 17.0 mm to (85.0, 34.2)
Connections:
- net Net-(J2-Pin_2) renamed GND1
- R14 pad 1: Net-(Q1-S-Pad1) -> Net-(Q2-S)
- R16 pad 1: Net-(Q1-S-Pad1) -> Net-(Q2-S)
- R17 pad 1: Net-(Q1-S-Pad1) -> Net-(Q2-S)
- R18 pad 1: Net-(Q1-S-Pad1) -> Net-(Q2-S)
- R19 pad 1: Net-(Q1-S-Pad1) -> Net-(Q2-S)
- R20 pad 1: Net-(Q1-S-Pad1) -> Net-(Q2-S)
- R21 pad 1: Net-(Q1-S-Pad1) -> Net-(Q2-S)
- R22 pad 1: Net-(Q1-S-Pad1) -> Net-(Q2-S)
- R23 pad 1: Net-(Q1-S-Pad1) -> Net-(Q2-S)
- R9 pad 1: Net-(Q1-S-Pad1) -> Net-(Q2-S)
- U1 pad 1: Net-(Q1-G) -> Net-(Q2-G)
- U2 pad 1: GND -> PACK-
- U2 pad 11: unconnected-(U2-P2.04-Pad11) -> /PGOOD21
- U2 pad 12: unconnected-(U2-P2.05-Pad12) -> /EN5
- U2 pad 13: unconnected-(U2-P2.03-Pad13) -> /PGOOD9
- U2 pad 16: GND -> PACK-
- U2 pad 27: GND -> PACK-
- U2 pad 38: unconnected-(U2-P2.06/CLK-Pad38) -> /EN9
- U2 pad 39: GND -> PACK-
- U2 pad 4: unconnected-(U2-P2.07-Pad4) -> /EN12
- U2 pad 8: unconnected-(U2-P2.02-Pad8) -> /PGOOD5
Routing:
- net 9VOUT: track 0.00 -> 0.74 mm
