File: BMS.kicad_sch (KiCad schematic)
At the start: 50 parts, among them J1 Conn_01x05_Pin, J10 XT90PB-F, J11 XT90PB-F, J12 XT90PB-F, J2 XT90PB-F, J3 Conn_01x02_Pin, J4 Conn_01x03_Pin, J5 XT90PB-F, J6 XT90PB-F, J7 XT90PB-F, J8 XT90PB-F, J9 XT90PB-F, Q2 IRLB3813PBF, U1 BQ76920PW

Commit message: Added Todo
Parts:
- C21, C22: footprint (none) -> Capacitor_SMD:C_0805_2012Metric_Pad1.18x1.45mm_HandSolder
Connections:
- net GND: no longer C11.2, C12.2, C21.2, C22.2, C4.2, C5.1, C6.2, C7.2, C8.2, C9.2
- net GND1: now reaches J2.1, R11.2, R14.2, R16.2, R17.2, R18.2, R19.2, R20.2, R21.2, R22.2, R23.2, R9.2, U1.3 (VSS)
- net GND1: now also C11.2, C12.2, C21.2, C22.2, C4.2, C5.1, C5.2, C6.2, C7.2, C8.2, C9.2, J1.1 (Pin_1), R5.2
Other:
- note added: "ADd uart"
- note added: "Add A/B Pins for new regs"
- note added: "Make sure connectors are right polarity"
- note added: "Separate connectors based on regs"
