File: PD.kicad_sch (KiCad schematic)
At the start: 33 parts, among them IC3 AOZ2261NQI-11, IC5 AOZ2261NQI-11

Commit message: Added Todo
Parts:
- added C28, C29, C30, C45, C46, C47: 22u, Capacitor_SMD:C_0805_2012Metric_Pad1.18x1.45mm_HandSolder, symbol Device:C
- added C31, C32, C38: 100n, Capacitor_SMD:C_0805_2012Metric_Pad1.18x1.45mm_HandSolder, symbol Device:C
- added C39, C40, C41: 10n, Capacitor_SMD:C_0805_2012Metric_Pad1.18x1.45mm_HandSolder, symbol Device:C
- added C42, C43, C44: 4u7, Capacitor_SMD:C_0805_2012Metric_Pad1.18x1.45mm_HandSolder, symbol Device:C
- added IC4, IC6, IC7: AOZ2261NQI-11, LIB_AOZ2261NQI-11:AOZ2261NQI11, symbol LIB_AOZ2261NQI-11:AOZ2261NQI-11
- added L4, L6, L7: 1u, Inductor_SMD:L_0805_2012Metric_Pad1.15x1.40mm_HandSolder, symbol Device:L
- added R34, R35, R36, R37, R42, R43: 100k, Resistor_SMD:R_0805_2012Metric_Pad1.20x1.40mm_HandSolder, symbol Device:R
- added R44: 190k, Resistor_SMD:R_0805_2012Metric_Pad1.20x1.40mm_HandSolder, symbol Device:R
- added R45, R47, R49: 10k, Resistor_SMD:R_0805_2012Metric_Pad1.20x1.40mm_HandSolder, symbol Device:R
- added R46: 140k, Resistor_SMD:R_0805_2012Metric_Pad1.20x1.40mm_HandSolder, symbol Device:R
- added R48: 75k, Resistor_SMD:R_0805_2012Metric_Pad1.20x1.40mm_HandSolder, symbol Device:R
- C13: renamed from C?; footprint (none) -> Capacitor_SMD:C_0805_2012Metric_Pad1.18x1.45mm_HandSolder
- C17, C18, C19, C20, C23, C24, C25, C26, C27, C33, C34, C35, C36, C37: footprint (none) -> Capacitor_SMD:C_0805_2012Metric_Pad1.18x1.45mm_HandSolder
- IC1: renamed from IC?; footprint AOZ2261NQI11 -> LIB_AOZ2261NQI-11:AOZ2261NQI11
- IC3, IC5: footprint AOZ2261NQI11 -> LIB_AOZ2261NQI-11:AOZ2261NQI11
- L2, L3, L5: footprint (none) -> Inductor_SMD:L_0805_2012Metric_Pad1.15x1.40mm_HandSolder
- R26, R27, R28, R29, R30, R31, R32, R33, R38, R39, R40, R41: footprint (none) -> Resistor_SMD:R_0805_2012Metric_Pad1.20x1.40mm_HandSolder
Connections:
- net +5V: now also C42.1, C43.1, C44.1, IC4.21 (VCC), IC6.21 (VCC), IC7.21 (VCC), R37.1, R42.1, R43.1
- net 12VOUT: now also C45.1, L4.2, R44.2
- net 5VOUT: now also C47.1, L7.2, R48.2
- net 9VOUT: now also C46.1, L6.2, R46.2
- net EN12: now also IC4.2 (EN/DISCHG)
- net EN5: now also IC7.2 (EN/DISCHG)
- net EN9: now also IC6.2 (EN/DISCHG)
- net FB12: now also IC4.5 (FB), R44.1, R45.2
- net FB5: now also IC7.5 (FB), R48.1, R49.2
- net FB9: now also IC6.5 (FB), R46.1, R47.2
- net GNDA: now also C39.2, C40.2, C41.2, C42.2, C43.2, C44.2, IC4.3 (MODE), IC4.4 (AGND), IC6.3 (MODE), IC6.4 (AGND), IC7.3 (MODE), IC7.4 (AGND), R45.1, R47.1, R49.1
- net GNDPWR: now also C28.2, C29.2, C30.2, C45.2, C46.2, C47.2, IC4.12 (PGND_1), IC4.13 (PGND_2), IC4.14 (PGND_3), IC4.15 (PGND_4), IC6.12 (PGND_1), IC6.13 (PGND_2), IC6.14 (PGND_3), IC6.15 (PGND_4), IC7.12 (PGND_1), IC7.13 (PGND_2), IC7.14 (PGND_3), IC7.15 (PGND_4)
- net LX12: now also C31.1, IC4.10 (LX_1), IC4.11 (LX_2), IC4.16 (LX_3), IC4.17 (LX_4), IC4.18 (LX_5), IC4.25 (LX_6), L4.1
- net LX5: now also C38.1, IC7.10 (LX_1), IC7.11 (LX_2), IC7.16 (LX_3), IC7.17 (LX_4), IC7.18 (LX_5), IC7.25 (LX_6), L7.1
- net LX9: now also C32.1, IC6.10 (LX_1), IC6.11 (LX_2), IC6.16 (LX_3), IC6.17 (LX_4), IC6.18 (LX_5), IC6.25 (LX_6), L6.1
- net PGOOD12: now also IC4.1 (PGOOD), R37.2
- net PGOOD5: now also IC7.1 (PGOOD), R43.2
- net PGOOD9 : now also IC6.1 (PGOOD), R42.2
- net VIN: now also C28.1, C29.1, C30.1, IC4.22 (IN_4), IC4.24 (IN_5), IC4.7 (IN_1), IC4.8 (IN_2), IC4.9 (IN_3), IC6.22 (IN_4), IC6.24 (IN_5), IC6.7 (IN_1), IC6.8 (IN_2), IC6.9 (IN_3), IC7.22 (IN_4), IC7.24 (IN_5), IC7.7 (IN_1), IC7.8 (IN_2), IC7.9 (IN_3), R34.2, R35.2, R36.2
- new net: C40.1, IC6.23 (SS)
- new net: C41.1, IC7.23 (SS)
- new net: IC6.6 (TON), R35.1
- new net: C32.2, IC6.20 (BST)
- new net: C38.2, IC7.20 (BST)
- new net: IC7.6 (TON), R36.1
- new net: IC4.6 (TON), R34.1
- new net: C31.2, IC4.20 (BST)
- new net: C39.1, IC4.23 (SS)
Other:
- moved on the sheet: C13, C17, C18, C19, C20, C23, C24, C25, C26, C27, C33, C34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
